Commit message: indy_eye  done

File: indy_description/urdf/indy.urdf.xacro (robot description, xacro)
@@ -7,5 +7,5 @@
     <!-- possible 'indy_type' values: indy7, indy12, indyrp2...-->
     <xacro:arg name="indy_type" default="indy7"/>
-    <xacro:arg name="indy_eye" default="false"/>
+    <xacro:arg name="indy_eye" default="true"/>
     <!-- parameters -->
     <xacro:arg name="prefix" default="" />

File: indy_description/urdf/indy_macro.xacro (robot description, xacro)
@@ -104,6 +104,7 @@
             <xacro:define_link link_name="link4" physic_name="link4" visual_name="link4" material="${material_1}" gazebo_material=""/>
             <xacro:define_link link_name="link5" physic_name="link5" visual_name="link5" material="${material_0}" gazebo_material=""/>
-            <xacro:if value="${indy_eye and not (indy_type == 'indyrp2' or indy_type == 'indyrp2_v2')}">
+            <xacro:if value="${indy_eye and indy_type == 'indy7'}">
                 <xacro:define_link link_name="link6" physic_name="link6" visual_name="link6_eye" material="${material_0}" gazebo_material=""/>
+                <link name="${prefix}indy_eye"/>
             </xacro:if>
             <xacro:unless value="${indy_eye and not (indy_type == 'indyrp2' or indy_type == 'indyrp2_v2')}">
@@ -194,4 +195,7 @@
             <xacro:define_joint joint_type="revolute" joint_index="joint4" parent_link="link4" child_link="link5"/>
             <xacro:define_joint joint_type="revolute" joint_index="joint5" parent_link="link5" child_link="link6"/>
+            <xacro:if value="${indy_eye and indy_type=='indy7'}">
+                <xacro:define_joint joint_type="fixed" joint_index="indy_eye" parent_link="link6" child_link="indy_eye"/>
+            </xacro:if>
             <xacro:if value="${indy_type == 'indyrp2' or indy_type == 'indyrp2_v2'}">
                 <xacro:define_joint joint_type="revolute" joint_index="joint6" parent_link="link6" child_link="link7"/>
@@ -211,4 +215,38 @@
         <!-- Add URDF transmission elements (for ros_control) -->
         <!-- <xacro:indy_transmission prefix="${prefix}" hw_interface="${transmission_hw_interface}" indy_type="${indy_type}"/> -->
+        <link name="${prefix}indy_eye_optical"/>
+        <joint name="${prefix}indy_eye_optical_joint" type="fixed">
+            <origin xyz="0 0 0" rpy="1.5707 -1.5707 0"/>
+            <parent link="${prefix}indy_eye"/>
+            <child link="${prefix}indy_eye_optical"/>
+        </joint>
+        <xacro:if value="${sim_gazebo and indy_eye}">
+            <gazebo reference="${prefix}indy_eye_optical">
+                <sensor name="indy_eye_camera" type="camera">
+                    <visualize>true</visualize>
+                    <always_on>true</always_on>
+                    <update_rate>30.0</update_rate>
+                    <camera name="eye_camera">
+                        <horizontal_fov>1.047</horizontal_fov>
+                        <image>
+                            <width>640</width>
+                            <height>480</height>
+                            <format>R8G8B8</format>
+                        </image>
+                        <clip>
+                            <near>0.05</near>
+                            <far>8.0</far>
+                        </clip>
+                    </camera>
+                    <plugin name="camera_controller" filename="libgazebo_ros_camera.so">
+                        <ros>
+                            <remapping>image_raw:=/camera/image_raw</remapping>
+                            <remapping>camera_info:=/camera/camera_info</remapping>
+                        </ros>
+                        <frame_name>${prefix}indy_eye_optical</frame_name>
+                    </plugin>
+                </sensor>
+            </gazebo>
+        </xacro:if>
     </xacro:macro>
 </robot>

Commit message: camera done :)

File: indy_description/urdf/indy.urdf.xacro (robot description, xacro)
@@ -39,6 +39,40 @@
         <origin xyz="0 0 0" rpy="0 0 0" />          <!-- position robot in the world -->
     </xacro:indy_robot>
+    <link name="$(arg prefix)indy_eye_optical"/>
+    <joint name="$(arg prefix)indy_eye_optical_joint" type="fixed">
+        <origin xyz="0 0 0" rpy="1.5707 -1.5707 -1.5707"/>
+        <!-- <origin xyz="0 0 0" rpy="0 0 0"/> -->
+        <!-- <origin xyz="0 0 0" rpy="1.5707 0 1.5707 "/> -->
+        <parent link="$(arg prefix)indy_eye"/>
+        <child link="$(arg prefix)indy_eye_optical"/>
+    </joint>
+    <gazebo reference="$(arg prefix)indy_eye_optical">
+		<sensor name="indy_eye_camera" type="camera">
+			<visualize>true</visualize>
+			<always_on>true</always_on>
+			<update_rate>30.0</update_rate>
+			<camera name="eye_camera">
+			<horizontal_fov>1.047</horizontal_fov>
+			<image>
+				<width>640</width>
+				<height>480</height>
+				<format>R8G8B8</format>
+			</image>
+			<clip>
+				<near>0.05</near>
+				<far>8.0</far>
+			</clip>
+			</camera>
+			<plugin name="camera_controller" filename="libgazebo_ros_camera.so">
+			<ros>
+				<remapping>image_raw:=/camera/image_raw</remapping>
+				<remapping>camera_info:=/camera/camera_info</remapping>
+			</ros>
+			<frame_name>$(arg prefix)indy_eye_optical</frame_name>
+			</plugin>
+		</sensor>
+	</gazebo>
     <xacro:if value="$(arg sim_gazebo)">
-        <gazebo reference="world"> </gazebo>
+        <gazebo reference="$(arg prefix)link0"> </gazebo>
         <gazebo>
             <plugin name="gazebo_ros2_control" filename="libgazebo_ros2_control.so" >

File: indy_description/urdf/indy_macro.xacro (robot description, xacro)
@@ -215,38 +215,4 @@
         <!-- Add URDF transmission elements (for ros_control) -->
         <!-- <xacro:indy_transmission prefix="${prefix}" hw_interface="${transmission_hw_interface}" indy_type="${indy_type}"/> -->
-        <link name="${prefix}indy_eye_optical"/>
-        <joint name="${prefix}indy_eye_optical_joint" type="fixed">
-            <origin xyz="0 0 0" rpy="1.5707 -1.5707 0"/>
-            <parent link="${prefix}indy_eye"/>
-            <child link="${prefix}indy_eye_optical"/>
-        </joint>
-        <xacro:if value="${sim_gazebo and indy_eye}">
-            <gazebo reference="${prefix}indy_eye_optical">
-                <sensor name="indy_eye_camera" type="camera">
-                    <visualize>true</visualize>
-                    <always_on>true</always_on>
-                    <update_rate>30.0</update_rate>
-                    <camera name="eye_camera">
-                        <horizontal_fov>1.047</horizontal_fov>
-                        <image>
-                            <width>640</width>
-                            <height>480</height>
-                            <format>R8G8B8</format>
-                        </image>
-                        <clip>
-                            <near>0.05</near>
-                            <far>8.0</far>
-                        </clip>
-                    </camera>
-                    <plugin name="camera_controller" filename="libgazebo_ros_camera.so">
-                        <ros>
-                            <remapping>image_raw:=/camera/image_raw</remapping>
-                            <remapping>camera_info:=/camera/camera_info</remapping>
-                        </ros>
-                        <frame_name>${prefix}indy_eye_optical</frame_name>
-                    </plugin>
-                </sensor>
-            </gazebo>
-        </xacro:if>
     </xacro:macro>
 </robot>

File: indy_description/urdf/indy_on_table.urdf.xacro (robot description, xacro)
@@ -4,4 +4,5 @@
     <xacro:include filename="$(find indy_description)/urdf/indy_macro.xacro"/>
     <xacro:include filename="$(find indy_description)/urdf/envs/table.xacro"/>
+    <xacro:include filename="$(find indy_description)/urdf/envs/camera.xacro"/>
     <!-- robot name parameter -->
     <xacro:arg name="name" default="indy"/>
@@ -30,5 +31,5 @@
         <parent link="table"/>
         <child  link="indy_mount_link"/>
-        <origin xyz="0.6 -0.4 0.2" rpy="0 0 1.57079632679"/>
+        <origin xyz="0.4 -0.2 0.2" rpy="0 0 1.57079632679"/>
     </joint>
     <!-- define robot -->
@@ -51,6 +52,47 @@
         <origin xyz="0 0 0" rpy="0 0 0" />          <!-- position robot in the world -->
     </xacro:indy_robot>
+    <link name="$(arg prefix)indy_eye_optical"/>
+    <joint name="$(arg prefix)indy_eye_optical_joint" type="fixed">
+        <!-- <origin xyz="0 0 0" rpy="1.5707 -1.5707 0"/> -->
+        <!-- <origin xyz="0 0 0" rpy="0 0 0"/> -->
+        <origin xyz="0 0 0" rpy="-1.5707 0 -1.5707 "/>
+        <parent link="$(arg prefix)indy_eye"/>
+        <child link="$(arg prefix)indy_eye_optical"/>
+    </joint>
+    <xacro:indy_eye_sensor
+        prefix="$(arg prefix)"
+        parent="$(arg prefix)indy_eye"
+        camType="depth"
+        >
+    </xacro:indy_eye_sensor>
+    <!-- <gazebo reference="$(arg prefix)indy_eye">
+		<sensor name="indy_eye_camera" type="camera">
+			<visualize>true</visualize>
+			<always_on>true</always_on>
+			<update_rate>30.0</update_rate>
+			<camera name="eye_camera">
+			<horizontal_fov>1.047</horizontal_fov>
+			<image>
+				<width>640</width>
+				<height>480</height>
+				<format>R8G8B8</format>
+			</image>
+			<clip>
+				<near>0.05</near>
+				<far>8.0</far>
+			</clip>
+			</camera>
+			<plugin name="camera_controller" filename="libgazebo_ros_camera.so">
+			<ros>
+				<remapping>image_raw:=/camera/image_raw</remapping>
+				<remapping>camera_info:=/camera/camera_info</remapping>
+			</ros>
+			<frame_name>$(arg prefix)indy_eye_optical</frame_name>
+			</plugin>
+		</sensor>
+	</gazebo> -->
     <xacro:if value="$(arg sim_gazebo)">
         <gazebo reference="world"> </gazebo>
+        <!-- <gazebo reference="indy_"> </gazebo> -->
         <gazebo>
             <plugin name="gazebo_ros2_control" filename="libgazebo_ros2_control.so" >

Commit message: workspace done:)

File: indy_description/urdf/indy.urdf.xacro (robot description, xacro)
@@ -39,40 +39,6 @@
         <origin xyz="0 0 0" rpy="0 0 0" />          <!-- position robot in the world -->
     </xacro:indy_robot>
-    <link name="$(arg prefix)indy_eye_optical"/>
-    <joint name="$(arg prefix)indy_eye_optical_joint" type="fixed">
-        <origin xyz="0 0 0" rpy="1.5707 -1.5707 -1.5707"/>
-        <!-- <origin xyz="0 0 0" rpy="0 0 0"/> -->
-        <!-- <origin xyz="0 0 0" rpy="1.5707 0 1.5707 "/> -->
-        <parent link="$(arg prefix)indy_eye"/>
-        <child link="$(arg prefix)indy_eye_optical"/>
-    </joint>
-    <gazebo reference="$(arg prefix)indy_eye_optical">
-		<sensor name="indy_eye_camera" type="camera">
-			<visualize>true</visualize>
-			<always_on>true</always_on>
-			<update_rate>30.0</update_rate>
-			<camera name="eye_camera">
-			<horizontal_fov>1.047</horizontal_fov>
-			<image>
-				<width>640</width>
-				<height>480</height>
-				<format>R8G8B8</format>
-			</image>
-			<clip>
-				<near>0.05</near>
-				<far>8.0</far>
-			</clip>
-			</camera>
-			<plugin name="camera_controller" filename="libgazebo_ros_camera.so">
-			<ros>
-				<remapping>image_raw:=/camera/image_raw</remapping>
-				<remapping>camera_info:=/camera/camera_info</remapping>
-			</ros>
-			<frame_name>$(arg prefix)indy_eye_optical</frame_name>
-			</plugin>
-		</sensor>
-	</gazebo>
     <xacro:if value="$(arg sim_gazebo)">
-        <gazebo reference="$(arg prefix)link0"> </gazebo>
+        <gazebo reference="world"> </gazebo>
         <gazebo>
             <plugin name="gazebo_ros2_control" filename="libgazebo_ros2_control.so" >

File: indy_description/urdf/indy_on_table.urdf.xacro (robot description, xacro)
@@ -54,6 +54,4 @@
     <link name="$(arg prefix)indy_eye_optical"/>
     <joint name="$(arg prefix)indy_eye_optical_joint" type="fixed">
-        <!-- <origin xyz="0 0 0" rpy="1.5707 -1.5707 0"/> -->
-        <!-- <origin xyz="0 0 0" rpy="0 0 0"/> -->
         <origin xyz="0 0 0" rpy="-1.5707 0 -1.5707 "/>
         <parent link="$(arg prefix)indy_eye"/>
@@ -63,36 +61,9 @@
         prefix="$(arg prefix)"
         parent="$(arg prefix)indy_eye"
-        camType="depth"
+        camType="camera"
         >
     </xacro:indy_eye_sensor>
-    <!-- <gazebo reference="$(arg prefix)indy_eye">
-		<sensor name="indy_eye_camera" type="camera">
-			<visualize>true</visualize>
-			<always_on>true</always_on>
-			<update_rate>30.0</update_rate>
-			<camera name="eye_camera">
-			<horizontal_fov>1.047</horizontal_fov>
-			<image>
-				<width>640</width>
-				<height>480</height>
-				<format>R8G8B8</format>
-			</image>
-			<clip>
-				<near>0.05</near>
-				<far>8.0</far>
-			</clip>
-			</camera>
-			<plugin name="camera_controller" filename="libgazebo_ros_camera.so">
-			<ros>
-				<remapping>image_raw:=/camera/image_raw</remapping>
-				<remapping>camera_info:=/camera/camera_info</remapping>
-			</ros>
-			<frame_name>$(arg prefix)indy_eye_optical</frame_name>
-			</plugin>
-		</sensor>
-	</gazebo> -->
     <xacro:if value="$(arg sim_gazebo)">
         <gazebo reference="world"> </gazebo>
-        <!-- <gazebo reference="indy_"> </gazebo> -->
         <gazebo>
             <plugin name="gazebo_ros2_control" filename="libgazebo_ros2_control.so" >
