Commit message: urdf problem maybe solved (camera link with no kinematics definition)

File: indy_description/urdf/indy.ros2_control.xacro (robot description, xacro)
@@ -21,8 +21,6 @@
                 <joint name="${prefix}${joint_index}">
                     <command_interface name="position">
-                        <!-- <param name="min">{-2*pi}</param>
-                        <param name="max">{2*pi}</param> -->
-                        <param name="min">-2*3.141592654</param>
-                        <param name="max">2*3.141592654</param>
+                        <param name="min">-6.3</param>
+                        <param name="max">6.3</param>
                     </command_interface>
                     <command_interface name="velocity">

File: indy_description/urdf/indy.urdf.xacro (robot description, xacro)
@@ -3,4 +3,5 @@
     <!-- import main macro -->
     <xacro:include filename="$(find indy_description)/urdf/indy_macro.xacro"/>
+    <xacro:include filename="$(find indy_description)/urdf/envs/camera.xacro"/>
     <!-- robot name parameter -->
     <xacro:arg name="name" default="indy"/>
@@ -39,4 +40,22 @@
         <origin xyz="0 0 0" rpy="0 0 0" />          <!-- position robot in the world -->
     </xacro:indy_robot>
+    <link name="$(arg prefix)indy_eye"/>
+    <joint name="$(arg prefix)indy_eye_joint" type="fixed">
+        <origin xyz="-0.08 0 0.06" rpy=" 0 -1.5707 0 "/>
+        <parent link="$(arg prefix)link6"/>
+        <child link="$(arg prefix)indy_eye"/>
+    </joint>
+    <link name="$(arg prefix)indy_eye_optical"/>
+    <joint name="$(arg prefix)indy_eye_optical_joint" type="fixed">
+        <origin xyz="0 0 0" rpy="-1.5707 0 -1.5707 "/>
+        <parent link="$(arg prefix)indy_eye"/>
+        <child link="$(arg prefix)indy_eye_optical"/>
+    </joint>
+    <xacro:indy_eye_sensor
+        prefix="$(arg prefix)"
+        parent="$(arg prefix)indy_eye"
+        camType="camera"
+        >
+    </xacro:indy_eye_sensor>
     <xacro:if value="$(arg sim_gazebo)">
         <gazebo reference="world"> </gazebo>

File: indy_description/urdf/indy_macro.xacro (robot description, xacro)
@@ -104,7 +104,6 @@
             <xacro:define_link link_name="link4" physic_name="link4" visual_name="link4" material="${material_1}" gazebo_material=""/>
             <xacro:define_link link_name="link5" physic_name="link5" visual_name="link5" material="${material_0}" gazebo_material=""/>
-            <xacro:if value="${indy_eye and indy_type == 'indy7'}">
+            <xacro:if value="${indy_eye and not (indy_type == 'indyrp2' or indy_type == 'indyrp2_v2')}">
                 <xacro:define_link link_name="link6" physic_name="link6" visual_name="link6_eye" material="${material_0}" gazebo_material=""/>
-                <link name="${prefix}indy_eye"/>
             </xacro:if>
             <xacro:unless value="${indy_eye and not (indy_type == 'indyrp2' or indy_type == 'indyrp2_v2')}">
@@ -195,7 +194,4 @@
             <xacro:define_joint joint_type="revolute" joint_index="joint4" parent_link="link4" child_link="link5"/>
             <xacro:define_joint joint_type="revolute" joint_index="joint5" parent_link="link5" child_link="link6"/>
-            <xacro:if value="${indy_eye and indy_type=='indy7'}">
-                <xacro:define_joint joint_type="fixed" joint_index="indy_eye" parent_link="link6" child_link="indy_eye"/>
-            </xacro:if>
             <xacro:if value="${indy_type == 'indyrp2' or indy_type == 'indyrp2_v2'}">
                 <xacro:define_joint joint_type="revolute" joint_index="joint6" parent_link="link6" child_link="link7"/>

File: indy_description/urdf/indy_on_table.urdf.xacro (robot description, xacro)
@@ -52,4 +52,10 @@
         <origin xyz="0 0 0" rpy="0 0 0" />          <!-- position robot in the world -->
     </xacro:indy_robot>
+    <link name="$(arg prefix)indy_eye"/>
+    <joint name="$(arg prefix)indy_eye_joint" type="fixed">
+        <origin xyz="-0.08 0 0.06" rpy=" 0 -1.5707 0 "/>
+        <parent link="$(arg prefix)link6"/>
+        <child link="$(arg prefix)indy_eye"/>
+    </joint>
     <link name="$(arg prefix)indy_eye_optical"/>
     <joint name="$(arg prefix)indy_eye_optical_joint" type="fixed">
