Commit message: realsense

File: indy_description/urdf/indy_on_table.urdf.xacro (robot description, xacro)
@@ -52,5 +52,5 @@
         <origin xyz="0 0 0" rpy="0 0 0" />          <!-- position robot in the world -->
     </xacro:indy_robot>
-    <link name="$(arg prefix)indy_eye"/>
+    <!-- <link name="$(arg prefix)indy_eye"/>
     <joint name="$(arg prefix)indy_eye_joint" type="fixed">
         <origin xyz="-0.08 0 0.06" rpy=" 0 -1.5707 0 "/>
@@ -63,9 +63,22 @@
         <parent link="$(arg prefix)indy_eye"/>
         <child link="$(arg prefix)indy_eye_optical"/>
+    </joint> -->
+    <link name="$(arg prefix)rs_eye"/>
+    <joint name="$(arg prefix)rs_eye_joint" type="fixed">
+        <!-- <origin xyz="0.06067 -0.02524 0.02966" rpy=" -1.6192 0.0100 0.2761 "/> -->
+        <origin xyz="0.06067 -0.02524 0.02966" rpy="0.0100 0.04805 1.8475"/>
+        <parent link="$(arg prefix)link6"/>
+        <child link="$(arg prefix)rs_eye"/>
+    </joint>
+    <link name="$(arg prefix)rs_eye_optical"/>
+    <joint name="$(arg prefix)rs_eye_optical_joint" type="fixed">
+        <origin xyz="0 0 0" rpy="-1.5707 0 -1.5707 "/>
+        <parent link="$(arg prefix)rs_eye"/>
+        <child link="$(arg prefix)rs_eye_optical"/>
     </joint>
     <xacro:indy_eye_sensor
         prefix="$(arg prefix)"
         parent="$(arg prefix)indy_eye"
-        camType="camera"
+        camType="depth"
         >
     </xacro:indy_eye_sensor>

Commit message: realsense 고육지책

File: indy_description/urdf/indy_on_table.urdf.xacro (robot description, xacro)
@@ -64,16 +64,17 @@
         <child link="$(arg prefix)indy_eye_optical"/>
     </joint> -->
-    <link name="$(arg prefix)rs_eye"/>
-    <joint name="$(arg prefix)rs_eye_joint" type="fixed">
+    <link name="$(arg prefix)indy_eye_optical"/>
+    <joint name="$(arg prefix)indy_eye__optical_joint" type="fixed">
         <!-- <origin xyz="0.06067 -0.02524 0.02966" rpy=" -1.6192 0.0100 0.2761 "/> -->
         <origin xyz="0.06067 -0.02524 0.02966" rpy="0.0100 0.04805 1.8475"/>
         <parent link="$(arg prefix)link6"/>
-        <child link="$(arg prefix)rs_eye"/>
+        <child link="$(arg prefix)indy_eye_optical"/>
     </joint>
-    <link name="$(arg prefix)rs_eye_optical"/>
-    <joint name="$(arg prefix)rs_eye_optical_joint" type="fixed">
-        <origin xyz="0 0 0" rpy="-1.5707 0 -1.5707 "/>
-        <parent link="$(arg prefix)rs_eye"/>
-        <child link="$(arg prefix)rs_eye_optical"/>
+    <link name="$(arg prefix)indy_eye"/>
+    <joint name="$(arg prefix)indy_eye_joint" type="fixed">
+        <!-- <origin xyz="0 0 0" rpy="-1.5707 0 -1.5707 "/> -->
+        <origin xyz="0 0 0" rpy="3.1415 -1.5707 -1.5707 "/>
+        <parent link="$(arg prefix)indy_eye_optical"/>
+        <child link="$(arg prefix)indy_eye"/>
     </joint>
     <xacro:indy_eye_sensor
