Commit message: 최신1

File: indy_description/urdf/envs/camera.xacro (robot description, xacro)
@@ -24,5 +24,5 @@
           <remapping>camera_info:=/camera/camera_info</remapping>
         </ros>
-        <frame_name>$(arg prefix)indy_eye_optical</frame_name>
+        <frame_name>${prefix}indy_eye_optical</frame_name>
         <xacro:if value="${camType == 'depth'}">
           <min_depth>0.05</min_depth>

File: indy_description/urdf/indy.urdf.xacro (robot description, xacro)
@@ -40,5 +40,5 @@
         <origin xyz="0 0 0" rpy="0 0 0" />          <!-- position robot in the world -->
     </xacro:indy_robot>
-    <link name="$(arg prefix)indy_eye"/>
+    <!-- <link name="$(arg prefix)indy_eye"/>
     <joint name="$(arg prefix)indy_eye_joint" type="fixed">
         <origin xyz="-0.08 0 0.06" rpy=" 0 -1.5707 0 "/>
@@ -51,4 +51,18 @@
         <parent link="$(arg prefix)indy_eye"/>
         <child link="$(arg prefix)indy_eye_optical"/>
+    </joint> -->
+    <link name="$(arg prefix)indy_eye_optical"/>
+    <joint name="$(arg prefix)indy_eye__optical_joint" type="fixed">
+        <!-- <origin xyz="0.06067 -0.02524 0.02966" rpy=" -1.6192 0.0100 0.2761 "/> -->
+        <origin xyz="0.06067 -0.02524 0.02966" rpy="0.0100 0.04805 1.8475"/>
+        <parent link="$(arg prefix)link6"/>
+        <child link="$(arg prefix)indy_eye_optical"/>
+    </joint>
+    <link name="$(arg prefix)indy_eye"/>
+    <joint name="$(arg prefix)indy_eye_joint" type="fixed">
+        <!-- <origin xyz="0 0 0" rpy="-1.5707 0 -1.5707 "/> -->
+        <origin xyz="0 0 0" rpy="3.1415 -1.5707 -1.5707 "/>
+        <parent link="$(arg prefix)indy_eye_optical"/>
+        <child link="$(arg prefix)indy_eye"/>
     </joint>
     <xacro:indy_eye_sensor

File: indy_description/urdf/indy_on_table.urdf.xacro (robot description, xacro)
@@ -31,5 +31,6 @@
         <parent link="table"/>
         <child  link="indy_mount_link"/>
-        <origin xyz="0.4 -0.2 0.2" rpy="0 0 1.57079632679"/>
+        <!-- <origin xyz="0.4 -0.2 0.2" rpy="0 0 1.57079632679"/> -->
+        <origin xyz="0.4 -0.2 0.2" rpy="0 0 3.141592"/>
     </joint>
     <!-- define robot -->
